File: eagle/revC/modules/module_HC05.brd (EAGLE design)
At the start: 24.1 x 32.8 mm, 40 parts

Commit message: Replaced modules with library parts
Parts:
- removed AIO0, AIO1, CLK, CSB, CTS, GND, GND1, GND2, MISO, MOSI, NC, PCCL, PCIN, PCOU, PCSY, PIO0, PIO1, PIO10, PIO11, PIO2, PIO3, PIO4, PIO5, PIO6, PIO7, PIO8, PIO9, RST, RTS, RXD, TXD, USB+, USB-, VCC: (no value), wirepad:SMD0,65-1,27
- added U$1: HC05, RadioShield:HC05
Connections:
- removed net UART_RX: LEFT1.3, RX.C, RXD.1
- removed net UART_TX: LEFT1.2, TX.C, TXD.1
- new net N$3: LEFT1.2, TX.C, U$1.TX
- new net N$4: LEFT1.3, RX.C, U$1.RX
- net GND: now also U$1.GND@1, U$1.GND@2, U$1.GND@3; no longer GND.1, GND1.1, GND2.1
- net VCC: no longer VCC.1
Routing:
- net N$4: track 0.00 -> 22.8 mm
- net UART_RX: track 22.8 -> 0.00 mm
- net N$3: track 0.00 -> 22.2 mm
- net UART_TX: track 22.1 -> 0.00 mm
- net VCC: track 34.1 -> 15.5 mm, vias 1 -> 0
Other:
- board text removed: "AIO0"
- board text removed: "AIO1"
- board text removed: "CLK"
- board text removed: "CSB"
- board text removed: "CTS"
- board text removed: "GND"
- board text removed: "GND2"
- board text removed: "MISO"
- board text removed: "MOSI"
- board text removed: "NC"
- board text removed: "PCCL"
- board text removed: "PCIN"
- board text removed: "PCOU"
- board text removed: "PCSY"
- board text removed: "PIO0"
- board text removed: "PIO1"
- board text removed: "PIO10"
- board text removed: "PIO11"
- board text removed: "PIO2"
- board text removed: "PIO3"
- board text removed: "PIO4"
- board text removed: "PIO5"
- board text removed: "PIO6"
- board text removed: "PIO7"
- board text removed: "PIO8"
- board text removed: "PIO9"
- board text removed: "RST"
- board text removed: "RTS"
- board text removed: "RXD"
- board text removed: "TXD"
- board text removed: "USB+"
- board text removed: "USB-"
- board text removed: "VCC"

Commit message: Fixed module name layers
Changed lines of the file:
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@@
 <wire x1="24.257" y1="26.543" x2="24.257" y2="0.127" width="0.254" layer="20"/>
 <wire x1="24.257" y1="0.127" x2="0.127" y2="0.127" width="0.254" layer="20"/>
-<text x="12.192" y="30.48" size="1.778" layer="51" ratio="15" rot="SR0" align="center">HC-05</text>
+<text x="12.192" y="30.48" size="1.778" layer="25" ratio="15" rot="SR0" align="center">HC-05</text>
 <text x="11.557" y="21.336" size="0.8128" layer="125" font="vector" ratio="12" rot="SR0" align="top-left">R1</text>
 <text x="11.557" y="25.4" size="0.8128" layer="125" font="vector" ratio="12" rot="SR0">R2</text>
