File: eagle/revC/modules/module_SX1262.brd (EAGLE design)
At the start: 24.1 x 32.8 mm, 4 parts, among them X1 734120110

Commit message: Fixed module name layers
Connections:
- net GND: no longer U$1.SW
Changed lines of the file:
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@@
 <wire x1="24.257" y1="26.543" x2="24.257" y2="0.127" width="0.254" layer="20"/>
 <wire x1="24.257" y1="0.127" x2="0.127" y2="0.127" width="0.254" layer="20"/>
-<text x="12.192" y="30.48" size="1.778" layer="51" ratio="15" rot="SR0" align="center">SX1262</text>
+<text x="12.192" y="30.48" size="1.778" layer="25" ratio="15" rot="SR0" align="center">SX1262</text>
 </plain>
 <attributes>
@@
 <contactref element="U$1" pad="GND@3"/>
 <contactref element="U$1" pad="GND@2"/>
-<contactref element="U$1" pad="SW"/>
 <contactref element="LEFT1" pad="10"/>
 <contactref element="X1" pad="S@2"/>
